Commit message: Created core URDF

File: description/robot_core.xacro (robot description, xacro)
@@ -26,5 +26,5 @@
     <link name="chassis">
         <visual>
-            <<origin xyz="0.107 0 0.025"/>
+            <origin xyz="0.107 0 0.025"/>
             <geometry>
                 <box size="0.214 0.15 0.05"/>
